File: hardware/board/elicio-v4.kicad_sch (KiCad schematic)
At the start: 62 parts, among them J2 202656-0021, J3 HDR-3-RA, J4 TC2030-NL, P1 SIG1, P2 SIG2, P3 REF, P4 CHARGE_VBUS, P5 CHARGE_GND, Q1 PMOS, Q2 NMOS, Q3 NMOS, Q4 NMOS, SW1 B3U-1000P, U1 ISP1807-LR, U2 ADS1292IRSMT, U3 BQ25100YFPR, U4 TLV71330PDQNR, U5 TPS7A0230PDQNR

Commit message: board(v4): W18 placement and locked pre-routes; not routed
elicio-v4.kicad_pcb is placed at W18 (W17 left too little B-side area for
the divider/interlock parts with via escape). 61 footprints, 0 keep-out
problems, every pad has a net. Locked pre-routes: SIG1/SIG2/REF strips to
R1-R3, the J3 branches on F (REF on B), charge nets across the joint on B
with the charger (U3) on B, nRESET round J4 to J4.6 and SW1, +VDD to J4.1,
the RF bridge and U1's inner VSS.

Schematic: R26 removed (P0.18 RESET has its own pull-up; firmware sets
UICR PSELRESET), pin map A on U1's east column, J3 pin order reversed so
the branches do not cross. ERC 0. Via rule 0.40/0.15 (JLC flex standard).
release.py takes --board.

State: DRC 0 errors, 125 unconnected items, 3 dangling warnings and 21
library-mismatch warnings (silk stripped). Not routed; no order outputs.

Co-Authored-By: Claude Opus 5.5 <noreply@anthropic.com>
Claude-Session: https://claude.ai/code/session_01RSpwhJjxHd7GLkEqrgCckN
Parts:
- removed R26: 10k, Resistor_SMD:R_0201_0603Metric, symbol Device:R
- C1: LCSC (none) -> C285104; MPN (none) -> 0201B152K500NT
- C10, C13, C16, C3, C4, C5: LCSC (none) -> C5142566; MPN (none) -> TCC0201X5R105K6R3ZT
- C11, C12, C15, C7: LCSC (none) -> C307380; MPN (none) -> CL03A104KO3NNNC
- C2: LCSC (none) -> C43380; MPN (none) -> 0201B103K500NT
- C6, C8, C9: LCSC (none) -> C15525; MPN (none) -> CL05A106MQ5NUNC
- P4, P5: footprint elicio:RING_PAD_D4.6_H2.7 -> elicio:RING_1S_D4.6_NPTH2.7
- Q1: value PMOS -> WPM3027-3; footprint Package_TO_SOT_SMD:SOT-723 -> Package_TO_SOT_SMD:SOT-883; LCSC (none) -> C240195; MPN (none) -> WPM3027-3/TR
- Q2, Q3, Q4: footprint Package_TO_SOT_SMD:SOT-723 -> Package_TO_SOT_SMD:SOT-883
- R11: LCSC (none) -> C4104700; MPN (none) -> ERJ-1GNF6801C
- R12: LCSC (none) -> C270341; MPN (none) -> 0201WMF6041TEE
- R13, R25, R27, R28, R5, R6, R7, R8: LCSC (none) -> C473048; MPN (none) -> 0201WMF1002TEE
- R14, R15, R16, R23, R24: LCSC (none) -> C270364; MPN (none) -> 0201WMF1003TEE
- R17, R20, R21, R4: LCSC (none) -> C473482; MPN (none) -> 0201WMF1004TEE
- R22: LCSC (none) -> C270365; MPN (none) -> 0201WMF1001TEE
- SW1: value B3U-1000P -> 1TS015A; footprint Button_Switch_SMD:SW_SPST_B3U-1000P -> elicio:SW_HRO_1TS015A; LCSC (none) -> C398746; MPN B3U-1000P -> 1TS015A-1200-0600-CT
- U3: footprint elicio:Texas_YFP0006 -> elicio:Texas_YFP0006_V4
- U4: value TLV71330PDQNR -> TLV71330PDQNT; LCSC (none) -> C3071062; MPN TLV71330PDQNR -> TLV71330PDQNT
Connections:
- net AFE_DRDY: now also U1.46 (P0.29/AIN5); no longer U1.6 (P0.26)
- net AFE_MISO: now also U1.32 (P0.08); no longer U1.46 (P0.29/AIN5)
- net AFE_MOSI: now also U1.36 (P0.05/AIN3); no longer U1.34 (P0.06)
- net AFE_RESET: now also U1.6 (P0.26); no longer U1.38 (P0.03/AIN1)
- net AFE_SCLK: now also U1.34 (P0.06); no longer U1.32 (P0.08)
- net AFE_START: now also U1.4 (P0.10/NFC2); no longer U1.44 (P0.30/AIN6)
- net CHG_MON: now also U1.44 (P0.30/AIN6); no longer U1.42 (P0.31/AIN7)
- net LED_EN: now also U1.38 (P0.03/AIN1); no longer U1.4 (P0.10/NFC2)
- net REF: now also J3.1 (Pin_1); no longer J3.3 (Pin_3)
- net SIG1: now also J3.3 (Pin_3); no longer J3.1 (Pin_1)
- net VBAT_SENSE: now also U1.42 (P0.31/AIN7); no longer U1.40 (P0.02/AIN0)
- net VBUS_DET: now also U1.40 (P0.02/AIN0); no longer U1.36 (P0.05/AIN3)
Other:
- title: Elicio board v4 (ISP1807, W17 body) -> Elicio board v4 (ISP1807, W18 body)

Commit message: wip(board v4): bench 220k on the J3 tab, VSS vias, folded tables; PCB not rebuilt, not routed
Design and generator changes only. hardware/board/elicio-v4.kicad_pcb is still
df6ae3a's board (GND in pieces, J3 Contact branches), so tests/test_board_v4.py
fails against it until the board is rebuilt and routed.

- v4_parts.py: J3 carries bench nets BENCH_SIG1/SIG2/REF behind their own 220k
  R31-R33 on the break-off tab (R7, Q97(d)); U1 VSS pads 14/16/18 on GND;
  consigned parts (U1, U5, J2) say CONSIGNED in the LCSC field.
- build_v4.py: tab u 20.1-33.4 x s 16-28, R31-R33 placed, AFE-side neck runs
  on F (s 20.40/21.15/21.90), two locked GND vias between U1 pads 14/16/18
  at u 6.70 (0.05 outside the RF band), --out for scratch builds.
- gen_v4_sch.py: bench nets in the Contact netclass; writes the .kicad_dru only
  if missing.
- v4_tables.py --folded: every courtyard, ring, strip root and tab root with
  cavity margins against the v4 target body; --pcb PATH.
- tests: Contact nets only on P1-P3/R1-R3, nothing Contact east of the island,
  bench header behind R31-R33, U1 VSS on GND.
- design note: §2, §3.1, §4.6, §5.4, §5.5, §7, §10.2, §11.1 updated. §9 still
  describes df6ae3a's state.

Co-Authored-By: Claude Fable 5.1 <noreply@anthropic.com>
Claude-Session: https://claude.ai/code/session_01UK16n13AdpykZ3bHg6Ep1F
Parts:
- added R31, R32, R33: 220k, Resistor_SMD:R_0402_1005Metric, symbol Device:R
- J2, U1, U5: LCSC (none) -> CONSIGNED
Connections:
- net AFE_IN1N: now also R32.1
- net AFE_IN1P: now also R31.1
- net GND: now also U1.14 (VSS), U1.16 (VSS), U1.18 (VSS)
- net REF: no longer J3.1 (Pin_1)
- net RLD_FB: now also R33.1
- net SIG1: no longer J3.3 (Pin_3)
- net SIG2: no longer J3.2 (Pin_2)
- new net BENCH_REF: J3.3 (Pin_3), R33.2
- new net BENCH_SIG1: J3.1 (Pin_1), R31.2
- new net BENCH_SIG2: J3.2 (Pin_2), R32.2
- no-connect marks 61 -> 58

Commit message: wip(board v4): refcheck t-0023 parts and pass-3 placement; PCB not rebuilt; NOT routed
- D1 PESD5V0L1UL on Nexperia's SOD882 land (pad 1 cathode on VBUS), moved to B at
  (14.60, 21.85) between R17 and C11.
- C11 VCAP2 1 uF at U2.27; C17 100 nF VREFP bypass beside C9.
- R34/R35 10k pull-downs on U2 GPIO1/GPIO2 (pins 26/25), on B under the east column.
- Q2-Q4 PMZ290UNE2 (C478155), pin 1 G, 2 S, 3 D.
- u2_core_pre_routes: U2 GND pads 10/13/24 tied to the exposed pad, one EP via to
  U4.5/U4.2/C8.2, VCAP2 to C11, GPIO1/GPIO2 hops to R34/R35.
- v4_gnd_split joins locked GND copper to the region of the pad it touches.

Schematic ERC 0. Board: router run 1 on this placement in progress, 17 nets still in
conflict at round 11. The committed PCB is still t-0014's; NOT routed.

Co-Authored-By: Claude Opus 5.5 <noreply@anthropic.com>
Claude-Session: https://claude.ai/code/session_01U4y3Vd9KrCnaj8gNYUDRvj
Parts:
- added C17: 100nF, Capacitor_SMD:C_0201_0603Metric, symbol Device:C
- added R34, R35: 10k, Resistor_SMD:R_0201_0603Metric, symbol Device:R
- C11: value 100nF -> 1uF; LCSC C307380 -> C5142566; MPN CL03A104KO3NNNC -> TCC0201X5R105K6R3ZT
- D1: footprint Diode_SMD:D_SOD-523 -> Diode_SMD:D_SOD-882
- Q2, Q3, Q4: value NMOS -> PMZ290UNE2; LCSC (none) -> C478155; MPN (none) -> PMZ290UNE2YL
Connections:
- net GND: now also C17.2, R34.2, R35.2
- net VREFP: now also C17.1
- net AFE_GPIO2: now reaches U2.25 (GPIO2)
- net AFE_GPIO2: now also R35.1
- net AFE_GPIO1: now reaches U2.26 (GPIO1)
- net AFE_GPIO1: now also R34.1
- no-connect marks 58 -> 56
