File: hardware/board/elicio-v4.kicad_pcb (KiCad board)
At the start: 2 copper layers, 31.1 x 55.2 mm, 67 parts, among them J2 202656-0021, J3 HDR-3-RA, J4 TC2030-NL, P1 SIG1, P2 SIG2, P3 REF, P4 CHARGE_VBUS, P5 CHARGE_GND, Q1 WPM3027-3, Q2 PMZ290UNE2, Q3 PMZ290UNE2, Q4 PMZ290UNE2, SW1 1TS015A, U1 ISP1807-LR, U2 ADS1292IRSMT, U3 BQ25100YFPR, U4 TLV71330PDQNT, U5 TPS7A0230PDQNR

Commit message: board(v4): add bias-rated charger bypasses and reroute release
Parts:
- added C18: 10uF, Capacitor_SMD:C_0402_1005Metric, B.Cu at (15.1, 20.7)
- added C19: 10uF, Capacitor_SMD:C_0402_1005Metric, F.Cu at (14.1, 34.2)
- C14: value 4.7uF -> 10uF
- C3: value 1uF -> 10uF; footprint Capacitor_SMD:C_0201_0603Metric -> Capacitor_SMD:C_0402_1005Metric; moved to F.Cu
- moved C3 2.40 mm to (14.4, 17.2)
- moved R17 0.75 mm to (13.7, 20.9)
Routing:
- net VBAT: track 25.0 -> 32.9 mm, vias 2 -> 3
- net GND: track 110.0 -> 114.0 mm, vias 17 -> 22
- net LED_EN: track 4.38 -> 6.49 mm
- net VBUS: track 48.9 -> 50.8 mm
- net TS: track 1.12 -> 2.46 mm, vias 1 -> 2
- net AFE_IN1P: track 30.0 -> 31.1 mm

Commit message: review(fab): align regulator value with stocked part and flag stale cost ranges
Parts:
- U4: value TLV71330PDQNT -> TLV71330PDQNR
Changed lines of the file:
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@@
 			)
 		)
-		(property "Value" "TLV71330PDQNT"
+		(property "Value" "TLV71330PDQNR"
 			(at 0 -1.5 0)
 			(layer "B.Fab")
